Commit message: added festo modules to the map and a reference link so they can be moved around

File: src/omtp_lecture1_2/urdf/omtp_factory.xacro (robot description, xacro)
@@ -1,91 +1,136 @@
 <?xml version="1.0" ?>
 <robot name="omtp_factory"
-  xmlns:xacro="http://www.ros.org/wiki/xacro">
-  <!-- ==================================================== -->
-  <!-- INITIAL SETUP OF WORLD LINK AND WORLD_INTERFACE LINK -->
-  <!-- ==================================================== -->
-  <!-- world -->
-  <link name="world" />
-  <!-- world_interface. Makes it convenient to move the whole environment according to the world origin -->
-  <link name="world_interface"/>
-  <!-- world<->world_interface joint -->
-  <joint name="world_interface_to_world" type="fixed">
-    <parent link="world" />
-    <child link="world_interface" />
-  </joint>
-  <!-- ==================================================== -->
-  <!-- Fib14 building -->
-  <!-- ==================================================== -->
-  <xacro:include filename="$(find aau_lab_ros_models)/urdf/fib14/fib14.urdf.xacro"/>
-  <xacro:fib14_urdf fib14_parent="world_interface"/>
-  <!-- ==================================================== -->
-  <!-- Panda robot -->
-  <!-- ==================================================== -->
-  <!-- Franka parameters -->
-  <xacro:arg name="arm_id_1" default="panda1"/>
-  <xacro:arg name="use_cylinder_collision_model" default="true"/>
-  <xacro:arg name="use_gazebo_sim" default="true"/>
-  <xacro:arg name="parent" default="robot1_pedestal_link"/>
-  <!-- Load panda arm and hand -->
-  <xacro:include filename="$(find franka_description)/robots/panda_arm.xacro" />
-  <xacro:include filename="$(find franka_description)/robots/hand.xacro"/>
-  <!-- Load gazebo control -->
-  <xacro:if value="$(arg use_gazebo_sim)">
-    <xacro:include filename="$(find franka_description)/robots/panda.gazebo.xacro"/>
-    <xacro:include filename="$(find franka_description)/robots/panda.control.xacro"/>
-  </xacro:if>
-  <!-- Panda 1 -->
-  <xacro:panda_arm xyz="0.05 0 0.95" rpy="0 0 0" connected_to="$(arg parent)" arm_id="$(arg arm_id_1)" safety_distance="0.03" use_cylinder_collision_model="$(arg use_cylinder_collision_model)"/>
-  <xacro:hand ns="$(arg arm_id_1)" rpy="0 0 ${-pi/4}" connected_to="$(arg arm_id_1)_link8" safety_distance="0.03" use_cylinder_collision_model="$(arg use_cylinder_collision_model)"/>
-  <xacro:arm_gazebo arm_id="$(arg arm_id_1)"/>
-  <xacro:arm_control arm_id="$(arg arm_id_1)"/>
-  <gazebo>
-    <plugin name="gazebo_ros_control" filename="libgazebo_ros_control.so"/>
-  </gazebo>
-  <!-- ==================================================== -->
-  <!-- Robot 1 pedestal -->
-  <!-- ==================================================== -->
-  <xacro:include filename="$(find external_ros_models)/urdf/robot_pedestal/robot_pedestal.urdf.xacro"/>
-  <xacro:robot_pedestal_urdf pedestal_prefix="robot1_" pedestal_parent="world_interface" pedestal_height="0.95">
-    <origin xyz="0.5 1.8 0.0" rpy="0 0 0"/>
-  </xacro:robot_pedestal_urdf>
-  <!-- ==================================================== -->
-  <!-- Bins -->
-  <!-- ==================================================== -->
-  <xacro:include filename="$(find external_ros_models)/urdf/bin/bin.urdf.xacro"/>
-  <xacro:bin_urdf prefix="bin_1"/>
-  <xacro:bin_urdf prefix="bin_2"/>
-  <xacro:bin_urdf prefix="bin_3"/>
-  <xacro:bin_urdf prefix="bin_4"/>
-  <xacro:bin_urdf prefix="bin_5"/>
-  <!-- Bin 1 -->
-  <joint name="bin_1_joint" type="fixed">
-    <parent link="world_interface" />
-    <child link="bin_1_base_link" />
-    <origin xyz="-0.3 1.2 0.0" rpy="0 0 0" />
-  </joint>
-  <!-- Bin 2 -->
-  <joint name="bin_2_joint" type="fixed">
-    <parent link="world_interface" />
-    <child link="bin_2_base_link" />
-    <origin xyz="-0.3 0.4 0.0" rpy="0 0 0" />
-  </joint>
-  <!-- Bin 3 -->
-  <joint name="bin_3_joint" type="fixed">
-    <parent link="world_interface" />
-    <child link="bin_3_base_link" />
-    <origin xyz="-0.3 -0.4 0.0" rpy="0 0 0" />
-  </joint>
-  <!-- Bin 4 -->
-  <joint name="bin_4_joint" type="fixed">
-    <parent link="world_interface" />
-    <child link="bin_4_base_link" />
-    <origin xyz="-0.3 -1.2 0.0" rpy="0 0 0" />
-  </joint>
-  <!-- Bin 5 -->
-  <joint name="bin_5_joint" type="fixed">
-    <parent link="world_interface" />
-    <child link="bin_5_base_link" />
-    <origin xyz="-0.3 -2.0 0.0" rpy="0 0 0" />
-  </joint>
+        xmlns:xacro="http://www.ros.org/wiki/xacro">
+        <!-- ==================================================== -->
+        <!-- INITIAL SETUP OF WORLD LINK AND WORLD_INTERFACE LINK -->
+        <!-- ==================================================== -->
+        <!-- world -->
+        <link name="world" />
+        <!-- world_interface. Makes it convenient to move the whole environment according to the world origin -->
+        <link name="world_interface"/>
+        <!-- world<->world_interface joint -->
+        <joint name="world_interface_to_world" type="fixed">
+                <parent link="world" />
+                <child link="world_interface" />
+        </joint>
+        <!-- ==================================================== -->
+        <!-- Fib14 building -->
+        <!-- ==================================================== -->
+        <xacro:include filename="$(find aau_lab_ros_models)/urdf/fib14/fib14.urdf.xacro"/>
+        <xacro:fib14_urdf fib14_parent="world_interface"/>
+        <!-- ==================================================== -->
+        <!-- Panda robot -->
+        <!-- ==================================================== -->
+        <!-- Franka parameters -->
+        <xacro:arg name="arm_id_1" default="panda1"/>
+        <xacro:arg name="use_cylinder_collision_model" default="true"/>
+        <xacro:arg name="use_gazebo_sim" default="true"/>
+        <xacro:arg name="parent" default="robot1_pedestal_link"/>
+        <!-- Load panda arm and hand -->
+        <xacro:include filename="$(find franka_description)/robots/panda_arm.xacro" />
+        <xacro:include filename="$(find franka_description)/robots/hand.xacro"/>
+        <!-- Load gazebo control -->
+        <xacro:if value="$(arg use_gazebo_sim)">
+                <xacro:include filename="$(find franka_description)/robots/panda.gazebo.xacro"/>
+                <xacro:include filename="$(find franka_description)/robots/panda.control.xacro"/>
+        </xacro:if>
+        <!-- Panda 1 -->
+        <xacro:panda_arm xyz="0.05 0 0.95" rpy="0 0 0" connected_to="$(arg parent)" arm_id="$(arg arm_id_1)" safety_distance="0.03" use_cylinder_collision_model="$(arg use_cylinder_collision_model)"/>
+        <xacro:hand ns="$(arg arm_id_1)" rpy="0 0 ${-pi/4}" connected_to="$(arg arm_id_1)_link8" safety_distance="0.03" use_cylinder_collision_model="$(arg use_cylinder_collision_model)"/>
+        <xacro:arm_gazebo arm_id="$(arg arm_id_1)"/>
+        <xacro:arm_control arm_id="$(arg arm_id_1)"/>
+        <gazebo>
+                <plugin name="gazebo_ros_control" filename="libgazebo_ros_control.so"/>
+        </gazebo>
+        <!-- ==================================================== -->
+        <!-- Robot 1 pedestal -->
+        <!-- ==================================================== -->
+        <xacro:include filename="$(find external_ros_models)/urdf/robot_pedestal/robot_pedestal.urdf.xacro"/>
+        <xacro:robot_pedestal_urdf pedestal_prefix="robot1_" pedestal_parent="world_interface" pedestal_height="0.95">
+                <origin xyz="0.5 1.8 0.0" rpy="0 0 0"/>
+        </xacro:robot_pedestal_urdf>
+        <!-- ==================================================== -->
+        <!-- Festo Modules -->
+        <!-- ==================================================== -->
+        <!-- Festo interface. Makes it convenient to move the whole Festo setup according to the world world interface-->
+        <link name="festo_interface"/>
+        <joint name="festo_to_world_interface" type="fixed">
+                <parent link="world_interface" />
+                <child link="festo_interface" />
+                <origin xyz="-2.0 3.0 0.0" rpy="0 0 0"/>
+        </joint>
+        <!-- Module 1 -->
+        <xacro:include filename="$(find aau_lab_ros_models)/urdf/festo_straight_module/festo_straight_module.urdf.xacro"/>
+        <xacro:festo_module_urdf module_prefix="module1_" festo_module_parent="festo_interface">
+                <origin xyz="1.0 0.0 0.0" rpy="0 0 0"/>
+        </xacro:festo_module_urdf>
+        <!-- Module 2 -->
+        <xacro:include filename="$(find aau_lab_ros_models)/urdf/festo_straight_module/festo_straight_module.urdf.xacro"/>
+        <xacro:festo_module_urdf module_prefix="module2_" festo_module_parent="festo_interface">
+                <origin xyz="1.0 1.2 0.0" rpy="0 0 0"/>
+        </xacro:festo_module_urdf>
+        <!-- T Module -->
+        <xacro:include filename="$(find aau_lab_ros_models)/urdf/festo_t_module/festo_t_module.urdf.xacro"/>
+        <xacro:festo_module_urdf module_prefix="moduleT_" festo_module_parent="festo_interface">
+                <origin xyz="1.0 2.4 0.0" rpy="0 0 0"/>
+        </xacro:festo_module_urdf>
+        <!-- Module 3 -->
+        <xacro:include filename="$(find aau_lab_ros_models)/urdf/festo_straight_module/festo_straight_module.urdf.xacro"/>
+        <xacro:festo_module_urdf module_prefix="module3_" festo_module_parent="festo_interface">
+                <origin xyz="0.0 2.4 0.0" rpy="0 0 ${pi/2}"/>
+        </xacro:festo_module_urdf>
+        <!-- Module 4 -->
+        <xacro:include filename="$(find aau_lab_ros_models)/urdf/festo_straight_module/festo_straight_module.urdf.xacro"/>
+        <xacro:festo_module_urdf module_prefix="module4_" festo_module_parent="festo_interface">
+                <origin xyz="-1.2 2.4 0.0" rpy="0 0 ${pi/2}"/>
+        </xacro:festo_module_urdf>
+        <!-- Module 5 -->
+        <xacro:include filename="$(find aau_lab_ros_models)/urdf/festo_straight_module/festo_straight_module.urdf.xacro"/>
+        <xacro:festo_module_urdf module_prefix="module5_" festo_module_parent="festo_interface">
+                <origin xyz="1.0 3.6 0.0" rpy="0 0 0"/>
+        </xacro:festo_module_urdf>
+        <!-- Module 6 -->
+        <xacro:include filename="$(find aau_lab_ros_models)/urdf/festo_straight_module/festo_straight_module.urdf.xacro"/>
+        <xacro:festo_module_urdf module_prefix="module6_" festo_module_parent="festo_interface">
+                <origin xyz="1.0 4.8 0.0" rpy="0 0 0"/>
+        </xacro:festo_module_urdf>
+        ====================================================
+                <!-- Bins -->
+        <!-- ==================================================== -->
+        <!-- <xacro:include filename="$(find external_ros_models)/urdf/bin/bin.urdf.xacro"/>
+        <xacro:bin_urdf prefix="bin_1"/>
+        <xacro:bin_urdf prefix="bin_2"/>
+        <xacro:bin_urdf prefix="bin_3"/>
+        <xacro:bin_urdf prefix="bin_4"/>
+        <xacro:bin_urdf prefix="bin_5"/>
+        Bin 1
+        <joint name="bin_1_joint" type="fixed">
+                <parent link="world_interface" />
+                <child link="bin_1_base_link" />
+                <origin xyz="-0.3 1.2 0.0" rpy="0 0 0" />
+        </joint>
+        Bin 2
+        <joint name="bin_2_joint" type="fixed">
+                <parent link="world_interface" />
+                <child link="bin_2_base_link" />
+                <origin xyz="-0.3 0.4 0.0" rpy="0 0 0" />
+        </joint>
+        Bin 3
+        <joint name="bin_3_joint" type="fixed">
+                <parent link="world_interface" />
+                <child link="bin_3_base_link" />
+                <origin xyz="-0.3 -0.4 0.0" rpy="0 0 0" />
+        </joint>
+        Bin 4
+        <joint name="bin_4_joint" type="fixed">
+                <parent link="world_interface" />
+                <child link="bin_4_base_link" />
+                <origin xyz="-0.3 -1.2 0.0" rpy="0 0 0" />
+        </joint>
+        Bin 5
+        <joint name="bin_5_joint" type="fixed">
+                <parent link="world_interface" />
+                <child link="bin_5_base_link" />
+                 <origin xyz="-0.3 -2.0 0.0" rpy="0 0 0" />
+        </joint> -->
 </robot>

Commit message: Inserted a second panda robot, and moved both to the correct location.

File: src/omtp_lecture1_2/urdf/omtp_factory.xacro (robot description, xacro)
@@ -20,5 +20,5 @@
         <xacro:fib14_urdf fib14_parent="world_interface"/>
         <!-- ==================================================== -->
-        <!-- Panda robot -->
+        <!-- Panda 1 robot -->
         <!-- ==================================================== -->
         <!-- Franka parameters -->
@@ -26,5 +26,5 @@
         <xacro:arg name="use_cylinder_collision_model" default="true"/>
         <xacro:arg name="use_gazebo_sim" default="true"/>
-        <xacro:arg name="parent" default="robot1_pedestal_link"/>
+        <xacro:arg name="panda1_parent" default="robot1_pedestal_link"/>
         <!-- Load panda arm and hand -->
         <xacro:include filename="$(find franka_description)/robots/panda_arm.xacro" />
@@ -36,5 +36,5 @@
         </xacro:if>
         <!-- Panda 1 -->
-        <xacro:panda_arm xyz="0.05 0 0.95" rpy="0 0 0" connected_to="$(arg parent)" arm_id="$(arg arm_id_1)" safety_distance="0.03" use_cylinder_collision_model="$(arg use_cylinder_collision_model)"/>
+        <xacro:panda_arm xyz="0.05 0 0.95" rpy="0 0 0" connected_to="$(arg panda1_parent)" arm_id="$(arg arm_id_1)" safety_distance="0.03" use_cylinder_collision_model="$(arg use_cylinder_collision_model)"/>
         <xacro:hand ns="$(arg arm_id_1)" rpy="0 0 ${-pi/4}" connected_to="$(arg arm_id_1)_link8" safety_distance="0.03" use_cylinder_collision_model="$(arg use_cylinder_collision_model)"/>
         <xacro:arm_gazebo arm_id="$(arg arm_id_1)"/>
@@ -48,5 +48,36 @@
         <xacro:include filename="$(find external_ros_models)/urdf/robot_pedestal/robot_pedestal.urdf.xacro"/>
         <xacro:robot_pedestal_urdf pedestal_prefix="robot1_" pedestal_parent="world_interface" pedestal_height="0.95">
-                <origin xyz="0.5 1.8 0.0" rpy="0 0 0"/>
+                <origin xyz="-1.6 3.0 0.0" rpy="0 0 0"/>
+        </xacro:robot_pedestal_urdf>
+        <!-- ==================================================== -->
+        <!-- Panda 2 robot -->
+        <!-- ==================================================== -->
+        <!-- Franka parameters -->
+        <xacro:arg name="arm_id_2" default="panda2"/>
+        <xacro:arg name="use_cylinder_collision_model" default="true"/>
+        <xacro:arg name="use_gazebo_sim" default="true"/>
+        <xacro:arg name="panda2_parent" default="robot2_pedestal_link"/>
+        <!-- Load panda arm and hand -->
+        <xacro:include filename="$(find franka_description)/robots/panda_arm.xacro" />
+        <xacro:include filename="$(find franka_description)/robots/hand.xacro"/>
+        <!-- Load gazebo control -->
+        <xacro:if value="$(arg use_gazebo_sim)">
+                <xacro:include filename="$(find franka_description)/robots/panda.gazebo.xacro"/>
+                <xacro:include filename="$(find franka_description)/robots/panda.control.xacro"/>
+        </xacro:if>
+        <!-- Panda 2 -->
+        <xacro:panda_arm xyz="0.05 0 0.95" rpy="0 0 0" connected_to="$(arg panda2_parent)" arm_id="$(arg arm_id_2)" safety_distance="0.03" use_cylinder_collision_model="$(arg use_cylinder_collision_model)"/>
+        <xacro:hand ns="$(arg arm_id_2)" rpy="0 0 ${-pi/4}" connected_to="$(arg arm_id_2)_link8" safety_distance="0.03" use_cylinder_collision_model="$(arg use_cylinder_collision_model)"/>
+        <xacro:arm_gazebo arm_id="$(arg arm_id_2)"/>
+        <xacro:arm_control arm_id="$(arg arm_id_2)"/>
+        <gazebo>
+                <plugin name="gazebo_ros_control" filename="libgazebo_ros_control.so"/>
+        </gazebo>
+        <!-- ==================================================== -->
+        <!-- Robot 2 pedestal -->
+        <!-- ==================================================== -->
+        <xacro:include filename="$(find external_ros_models)/urdf/robot_pedestal/robot_pedestal.urdf.xacro"/>
+        <xacro:robot_pedestal_urdf pedestal_prefix="robot2_" pedestal_parent="world_interface" pedestal_height="0.95">
+                <origin xyz="-1.6 6.6 0.0" rpy="0 0 0"/>
         </xacro:robot_pedestal_urdf>
         <!-- ==================================================== -->
@@ -96,5 +127,5 @@
         </xacro:festo_module_urdf>
         ====================================================
-                <!-- Bins -->
+                                                                                                                                                                                                                <!-- Bins -->
         <!-- ==================================================== -->
         <!-- <xacro:include filename="$(find external_ros_models)/urdf/bin/bin.urdf.xacro"/>
