Commit message: Got the manipulators to stand up straight in gazebo. So i attached the arm controllers to gazebo.

File: src/omtp_lecture1_2/urdf/omtp.urdf (robot description, URDF)
Before this commit: robot omtp_factory, 24 links, 23 joints
Links:
- added link panda2_hand, mass 0.48; collision cylinder length=0.1 radius=0.05; collision cylinder length=0.1 radius=0.07
- added link panda2_leftfinger, mass 0.1; visual mesh filename=package://franka_description/meshes/visual/finger.dae
- added link panda2_link0, mass 3.06; collision cylinder length=0.2830 radius=0.09; collision sphere radius=0.09
- added link panda2_link1, mass 2.34; collision cylinder length=0.2830 radius=0.09; collision sphere radius=0.09
- added link panda2_link2, mass 2.36; collision cylinder length=0.12 radius=0.09; collision sphere radius=0.09
- added link panda2_link3, mass 2.38; collision cylinder length=0.15 radius=0.09; collision sphere radius=0.09
- added link panda2_link4, mass 2.43; collision cylinder length=0.12 radius=0.09; collision sphere radius=0.09
- added link panda2_link5, mass 3.5; collision cylinder length=0.1 radius=0.09; collision cylinder length=0.14 radius=0.055
- added link panda2_link6, mass 1.47; collision cylinder length=0.08 radius=0.08; collision sphere radius=0.08
- added link panda2_link7, mass 0.45; collision cylinder length=0.14 radius=0.07; collision sphere radius=0.07
- added link panda2_link8, mass 0.0; collision cylinder length=0.01 radius=0.06; collision sphere radius=0.06
- added link panda2_rightfinger, mass 0.1; visual mesh filename=package://franka_description/meshes/visual/finger.dae
- added link robot2_pedestal_link, mass 500; collision box size=0.3 0.3 0.95; visual box size=0.3 0.3 0.95
Joints:
- added joint panda2_finger_joint1: type prismatic, parent panda2_hand, child panda2_leftfinger, origin xyz=0 0 0.0584 rpy=0 0 0, axis 0 1 0, limit lower=0.0 upper=0.04 effort=150 velocity=0.2
- added joint panda2_finger_joint2: type prismatic, parent panda2_hand, child panda2_rightfinger, origin xyz=0 0 0.0584 rpy=0 0 0, axis 0 -1 0, limit lower=0.0 upper=0.04 effort=150 velocity=0.2
- added joint panda2_hand_joint: type fixed, parent panda2_link8, child panda2_hand, origin xyz=0 0 0 rpy=0 0 -0.7853981633974483
- added joint panda2_joint1: type revolute, parent panda2_link0, child panda2_link1, origin xyz=0 0 0.333 rpy=0 0 0, axis 0 0 1, limit lower=-2.8973 upper=2.8973 effort=87 velocity=2.175
- added joint panda2_joint2: type revolute, parent panda2_link1, child panda2_link2, origin xyz=0 0 0 rpy=-1.5707963267948966 0 0, axis 0 0 1, limit lower=-1.7628 upper=1.7628 effort=87 velocity=2.175
- added joint panda2_joint3: type revolute, parent panda2_link2, child panda2_link3, origin xyz=0 -0.316 0 rpy=1.5707963267948966 0 0, axis 0 0 1, limit lower=-2.8973 upper=2.8973 effort=87 velocity=2.175
- added joint panda2_joint4: type revolute, parent panda2_link3, child panda2_link4, origin xyz=0.0825 0 0 rpy=1.5707963267948966 0 0, axis 0 0 1, limit lower=-3.0718 upper=-0.0698 effort=87 velocity=2.175
- added joint panda2_joint5: type revolute, parent panda2_link4, child panda2_link5, origin xyz=-0.0825 0.384 0 rpy=-1.5707963267948966 0 0, axis 0 0 1, limit lower=-2.8973 upper=2.8973 effort=12 velocity=2.61
- added joint panda2_joint6: type revolute, parent panda2_link5, child panda2_link6, origin xyz=0 0 0 rpy=1.5707963267948966 0 0, axis 0 0 1, limit lower=-0.0175 upper=3.7525 effort=12 velocity=2.61
- added joint panda2_joint7: type revolute, parent panda2_link6, child panda2_link7, origin xyz=0.088 0 0 rpy=1.5707963267948966 0 0, axis 0 0 1, limit lower=-2.8973 upper=2.8973 effort=12 velocity=2.61
- added joint panda2_joint8: type fixed, parent panda2_link7, child panda2_link8, origin xyz=0 0 0.107 rpy=0 0 0, axis 0 0 0
- added joint panda2_virtual_joint: type fixed, parent robot2_pedestal_link, child panda2_link0, origin xyz=0.05 0 0.95 rpy=0 0 0
- added joint robot2_pedestal_joint: type fixed, parent world_interface, child robot2_pedestal_link, origin xyz=-1.6 6.6 0.0 rpy=0 0 0
- joint robot1_pedestal_joint: origin xyz=0.5 1.8 0.0 rpy=0 0 0 -> xyz=-1.6 3.0 0.0 rpy=0 0 0

File: src/omtp_lecture1_2/urdf/omtp_factory.xacro (robot description, xacro)
@@ -55,6 +55,4 @@
         <!-- Franka parameters -->
         <xacro:arg name="arm_id_2" default="panda2"/>
-        <xacro:arg name="use_cylinder_collision_model" default="true"/>
-        <xacro:arg name="use_gazebo_sim" default="true"/>
         <xacro:arg name="panda2_parent" default="robot2_pedestal_link"/>
         <!-- Load panda arm and hand -->
@@ -126,6 +124,6 @@
                 <origin xyz="1.0 4.8 0.0" rpy="0 0 0"/>
         </xacro:festo_module_urdf>
-        ====================================================
-                                                                                                                                                                                                                <!-- Bins -->
+        <!-- ==================================================== -->
+        <!-- Bins -->
         <!-- ==================================================== -->
         <!-- <xacro:include filename="$(find external_ros_models)/urdf/bin/bin.urdf.xacro"/>
