Commit message: Synchronized gazebo with rviz, so planning is done in gazebo.

File: src/lecture2_single_panda_moveit_config/config/omtp_factory.ros2_control.xacro (robot description, xacro)
@@ -1,75 +1,80 @@
 <?xml version="1.0"?>
 <robot xmlns:xacro="http://www.ros.org/wiki/xacro">
-    <xacro:macro name="omtp_factory_ros2_control" params="name initial_positions_file">
-        <xacro:property name="initial_positions" value="${load_yaml(initial_positions_file)['initial_positions']}"/>
-        <ros2_control name="${name}" type="system">
-            <hardware>
-                <!-- By default, set up controllers for simulation. This won't work on real hardware -->
-                <plugin>mock_components/GenericSystem</plugin>
-            </hardware>
-            <joint name="panda1_joint1">
-                <command_interface name="position"/>
-                <state_interface name="position">
-                  <param name="initial_value">${initial_positions['panda1_joint1']}</param>
-                </state_interface>
-                <state_interface name="velocity"/>
-            </joint>
-            <joint name="panda1_joint2">
-                <command_interface name="position"/>
-                <state_interface name="position">
-                  <param name="initial_value">${initial_positions['panda1_joint2']}</param>
-                </state_interface>
-                <state_interface name="velocity"/>
-            </joint>
-            <joint name="panda1_joint3">
-                <command_interface name="position"/>
-                <state_interface name="position">
-                  <param name="initial_value">${initial_positions['panda1_joint3']}</param>
-                </state_interface>
-                <state_interface name="velocity"/>
-            </joint>
-            <joint name="panda1_joint4">
-                <command_interface name="position"/>
-                <state_interface name="position">
-                  <param name="initial_value">${initial_positions['panda1_joint4']}</param>
-                </state_interface>
-                <state_interface name="velocity"/>
-            </joint>
-            <joint name="panda1_joint5">
-                <command_interface name="position"/>
-                <state_interface name="position">
-                  <param name="initial_value">${initial_positions['panda1_joint5']}</param>
-                </state_interface>
-                <state_interface name="velocity"/>
-            </joint>
-            <joint name="panda1_joint6">
-                <command_interface name="position"/>
-                <state_interface name="position">
-                  <param name="initial_value">${initial_positions['panda1_joint6']}</param>
-                </state_interface>
-                <state_interface name="velocity"/>
-            </joint>
-            <joint name="panda1_joint7">
-                <command_interface name="position"/>
-                <state_interface name="position">
-                  <param name="initial_value">${initial_positions['panda1_joint7']}</param>
-                </state_interface>
-                <state_interface name="velocity"/>
-            </joint>
-            <joint name="panda1_finger_joint1">
-                <command_interface name="position"/>
-                <state_interface name="position">
-                  <param name="initial_value">${initial_positions['panda1_finger_joint1']}</param>
-                </state_interface>
-                <state_interface name="velocity"/>
-            </joint>
-            <joint name="panda1_finger_joint2">
-                <command_interface name="position"/>
-                <state_interface name="position">
-                  <param name="initial_value">${initial_positions['panda1_finger_joint2']}</param>
-                </state_interface>
-                <state_interface name="velocity"/>
-            </joint>
-        </ros2_control>
-    </xacro:macro>
+  <xacro:macro name="omtp_factory_ros2_control" params="name initial_positions_file">
+    <xacro:property name="initial_positions" value="${load_yaml(initial_positions_file)['initial_positions']}"/>
+    <ros2_control name="${name}" type="system">
+      <hardware>
+        <!-- By default, set up controllers for simulation. This won't work on real hardware -->
+        <plugin>gazebo_ros2_control/GazeboSystem</plugin>
+      </hardware>
+      <joint name="panda1_joint1">
+        <command_interface name="position"/>
+        <state_interface name="position">
+          <param name="initial_value">${initial_positions['panda1_joint1']}</param>
+        </state_interface>
+        <state_interface name="velocity"/>
+      </joint>
+      <joint name="panda1_joint2">
+        <command_interface name="position"/>
+        <state_interface name="position">
+          <param name="initial_value">${initial_positions['panda1_joint2']}</param>
+        </state_interface>
+        <state_interface name="velocity"/>
+      </joint>
+      <joint name="panda1_joint3">
+        <command_interface name="position"/>
+        <state_interface name="position">
+          <param name="initial_value">${initial_positions['panda1_joint3']}</param>
+        </state_interface>
+        <state_interface name="velocity"/>
+      </joint>
+      <joint name="panda1_joint4">
+        <command_interface name="position"/>
+        <state_interface name="position">
+          <param name="initial_value">${initial_positions['panda1_joint4']}</param>
+        </state_interface>
+        <state_interface name="velocity"/>
+      </joint>
+      <joint name="panda1_joint5">
+        <command_interface name="position"/>
+        <state_interface name="position">
+          <param name="initial_value">${initial_positions['panda1_joint5']}</param>
+        </state_interface>
+        <state_interface name="velocity"/>
+      </joint>
+      <joint name="panda1_joint6">
+        <command_interface name="position"/>
+        <state_interface name="position">
+          <param name="initial_value">${initial_positions['panda1_joint6']}</param>
+        </state_interface>
+        <state_interface name="velocity"/>
+      </joint>
+      <joint name="panda1_joint7">
+        <command_interface name="position"/>
+        <state_interface name="position">
+          <param name="initial_value">${initial_positions['panda1_joint7']}</param>
+        </state_interface>
+        <state_interface name="velocity"/>
+      </joint>
+      <joint name="panda1_finger_joint1">
+        <command_interface name="position"/>
+        <state_interface name="position">
+          <param name="initial_value">${initial_positions['panda1_finger_joint1']}</param>
+        </state_interface>
+        <state_interface name="velocity"/>
+      </joint>
+      <joint name="panda1_finger_joint2">
+        <command_interface name="position"/>
+        <state_interface name="position">
+          <param name="initial_value">${initial_positions['panda1_finger_joint2']}</param>
+        </state_interface>
+        <state_interface name="velocity"/>
+      </joint>
+    </ros2_control>
+    <gazebo>
+      <plugin name="gazebo_ros2_control" filename="libgazebo_ros2_control.so">
+        <parameters>$(find lecture2_single_panda_moveit_config)/config/ros2_controllers.yaml</parameters>
+      </plugin>
+    </gazebo>
+  </xacro:macro>
 </robot>

File: src/lecture2_single_panda_moveit_config/config/omtp_factory.urdf.xacro (robot description, xacro)
@@ -6,4 +6,4 @@
     <!-- Import control_xacro -->
     <xacro:include filename="omtp_factory.ros2_control.xacro" />
-    <xacro:omtp_factory_ros2_control name="FakeSystem" initial_positions_file="$(arg initial_positions_file)"/>
+    <xacro:omtp_factory_ros2_control name="GazeboSystem" initial_positions_file="$(arg initial_positions_file)"/>
 </robot>

File: src/omtp_lecture1_2/urdf/omtp.urdf (robot description, URDF)
Before this commit: robot omtp_factory, 37 links, 36 joints
Links:
- removed link panda2_hand
- removed link panda2_leftfinger
- removed link panda2_link0
- removed link panda2_link1
- removed link panda2_link2
- removed link panda2_link3
- removed link panda2_link4
- removed link panda2_link5
- removed link panda2_link6
- removed link panda2_link7
- removed link panda2_link8
- removed link panda2_rightfinger
- removed link robot2_pedestal_link
Joints:
- removed joint panda2_finger_joint1
- removed joint panda2_finger_joint2
- removed joint panda2_hand_joint
- removed joint panda2_joint1
- removed joint panda2_joint2
- removed joint panda2_joint3
- removed joint panda2_joint4
- removed joint panda2_joint5
- removed joint panda2_joint6
- removed joint panda2_joint7
- removed joint panda2_joint8
- removed joint panda2_virtual_joint
- removed joint robot2_pedestal_joint

File: src/omtp_lecture1_2/urdf/omtp_factory.xacro (robot description, xacro)
@@ -40,7 +40,7 @@
         <xacro:arm_gazebo arm_id="$(arg arm_id_1)"/>
         <xacro:arm_control arm_id="$(arg arm_id_1)"/>
-        <gazebo>
-                <plugin name="gazebo_ros_control" filename="libgazebo_ros_control.so"/>
-        </gazebo>
+        <!-- <gazebo>
+                <plugin name="gazebo_ros2_control" filename="libgazebo_ros2_control.so"/>
+        </gazebo> -->
         <!-- ==================================================== -->
         <!-- Robot 1 pedestal -->
@@ -54,29 +54,26 @@
         <!-- ==================================================== -->
         <!-- Franka parameters -->
-        <xacro:arg name="arm_id_2" default="panda2"/>
-        <xacro:arg name="panda2_parent" default="robot2_pedestal_link"/>
+        <!-- <xacro:arg name="arm_id_2" default="panda2"/>
+        <xacro:arg name="panda2_parent" default="robot2_pedestal_link"/> -->
         <!-- Load panda arm and hand -->
-        <xacro:include filename="$(find franka_description)/robots/panda_arm.xacro" />
-        <xacro:include filename="$(find franka_description)/robots/hand.xacro"/>
+        <!-- <xacro:include filename="$(find franka_description)/robots/panda_arm.xacro" />
+        <xacro:include filename="$(find franka_description)/robots/hand.xacro"/> -->
         <!-- Load gazebo control -->
-        <xacro:if value="$(arg use_gazebo_sim)">
+        <!-- <xacro:if value="$(arg use_gazebo_sim)">
                 <xacro:include filename="$(find franka_description)/robots/panda.gazebo.xacro"/>
                 <xacro:include filename="$(find franka_description)/robots/panda.control.xacro"/>
-        </xacro:if>
+        </xacro:if> -->
         <!-- Panda 2 -->
-        <xacro:panda_arm xyz="0.05 0 0.95" rpy="0 0 0" connected_to="$(arg panda2_parent)" arm_id="$(arg arm_id_2)" safety_distance="0.03" use_cylinder_collision_model="$(arg use_cylinder_collision_model)"/>
+        <!-- <xacro:panda_arm xyz="0.05 0 0.95" rpy="0 0 0" connected_to="$(arg panda2_parent)" arm_id="$(arg arm_id_2)" safety_distance="0.03" use_cylinder_collision_model="$(arg use_cylinder_collision_model)"/>
         <xacro:hand ns="$(arg arm_id_2)" rpy="0 0 ${-pi/4}" connected_to="$(arg arm_id_2)_link8" safety_distance="0.03" use_cylinder_collision_model="$(arg use_cylinder_collision_model)"/>
         <xacro:arm_gazebo arm_id="$(arg arm_id_2)"/>
-        <xacro:arm_control arm_id="$(arg arm_id_2)"/>
-        <gazebo>
-                <plugin name="gazebo_ros_control" filename="libgazebo_ros_control.so"/>
-        </gazebo>
+        <xacro:arm_control arm_id="$(arg arm_id_2)"/> -->
         <!-- ==================================================== -->
         <!-- Robot 2 pedestal -->
         <!-- ==================================================== -->
-        <xacro:include filename="$(find external_ros_models)/urdf/robot_pedestal/robot_pedestal.urdf.xacro"/>
+        <!-- <xacro:include filename="$(find external_ros_models)/urdf/robot_pedestal/robot_pedestal.urdf.xacro"/>
         <xacro:robot_pedestal_urdf pedestal_prefix="robot2_" pedestal_parent="world_interface" pedestal_height="0.95">
                 <origin xyz="-1.6 6.6 0.0" rpy="0 0 0"/>
-        </xacro:robot_pedestal_urdf>
+        </xacro:robot_pedestal_urdf> -->
         <!-- ==================================================== -->
         <!-- Festo Modules -->

Commit message: Removed deprecated load_yaml().

File: src/lecture2_single_panda_moveit_config/config/omtp_factory.ros2_control.xacro (robot description, xacro)
@@ -2,5 +2,5 @@
 <robot xmlns:xacro="http://www.ros.org/wiki/xacro">
   <xacro:macro name="omtp_factory_ros2_control" params="name initial_positions_file">
-    <xacro:property name="initial_positions" value="${load_yaml(initial_positions_file)['initial_positions']}"/>
+    <xacro:property name="initial_positions" value="${xacro.load_yaml(initial_positions_file)['initial_positions']}"/>
     <ros2_control name="${name}" type="system">
       <hardware>
